File: H7PI/H7PI.sch (KiCad schematic (older format))
At the start: 52 parts, among them J1 XKTF-015-N, J10 DNP, J2 Header_2x10, J3 microUSB, J4 AFC07-S24ECA-00, J5 Header_2x20, J6 microUSB, J7 Header_1x2, J8 Header_1x1, J9 Header_1x1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

Commit message: v0.4 add pin info to bottom silk change pin name to Dx,Ax.
Signed-off-by: fuhua-chen <fuhua-chen@outlook.com>
Parts:
- removed J10: DNP, PinHeader_1x02_P2.54mm_Vertical, symbol connector:Header_1x2
- J2: value Header_2x10 -> Header_2x11; footprint PinHeader_2x10_P2.54mm_Vertical -> PinHeader_2x11_P2.54mm_Vertical; symbol connector:Header_2x10 -> connector:Header_2x11
Connections:
- net USB_N: now also J2.21
- net USB_P: now also J2.22
- net IO1 renamed D8
- net IO10 renamed D17
- net IO11 renamed D18
- net IO12 renamed D19
- net IO13 renamed D20
- net IO14 renamed D21
- net IO15 renamed D22
- net IO16 renamed D23
- net IO2 renamed D9
- net IO3 renamed D10
- net IO4 renamed D11
- net IO5 renamed D12
- net IO6 renamed D13
- net IO7 renamed D14
- net IO8 renamed D15
- net IO9 renamed D16
- net PI_CE0 renamed CE0
- net PI_CE1 renamed CE1
- net PI_GPIO0 renamed D0
- net PI_GPIO1 renamed D1
- net PI_GPIO2 renamed D2
- net PI_GPIO21 renamed A0
- net PI_GPIO22 renamed A1
- net PI_GPIO23 renamed A2
- net PI_GPIO24 renamed A3
- net PI_GPIO25 renamed A4
- net PI_GPIO26 renamed A5
- net PI_GPIO27 renamed A6
- net PI_GPIO28 renamed A7
- net PI_GPIO29 renamed D29
- net PI_GPIO3 renamed D3
- net PI_GPIO4 renamed D4
- net PI_GPIO5 renamed D5
- net PI_GPIO6 renamed D6
- net PI_GPIO7 renamed D7
- net PI_MISO renamed MISO
- net PI_MOSI renamed MOSI
- net PI_RXD renamed RX0
- net PI_SCK renamed SCK
- net PI_SCL0 renamed SCL0
- net PI_SCL1 renamed SCL1
- net PI_SDA0 renamed SDA0
- net PI_SDA1 renamed SDA1
- net PI_TXD renamed TX0
